Commit message: Update hexapod.urdf.xacro

File: src/hexapod_ws/description/hexapod.urdf.xacro (robot description, xacro)
@@ -255,5 +255,5 @@
     <parent link="core"/>
     <child  link="camera"/>
-    <origin xyz="0.045842 -0.000288 0.11141" rpy="-0.00418892 0 0.00038394"/>
+    <origin xyz="0.050842 -0.000288 0.11141" rpy="-0.00418892 0 0.00038394"/>
   </joint>
   <gazebo reference="camera">
